File: KiCad Schematic and PCB/Rocket Club V1 Schematic I2C 7.kicad_sch (KiCad schematic)
At the start: 32 parts, among them IC1 STM32H573RIT6, IC2 BNO085, IC4 MT29F1G08ABAEAWP_E, J1 USB4135-GF-A_REVA, U1 H3LIS100DLTR, U3 MAX-M8W-0

Commit message: Updated schematic, not fully done but majority done
Parts:
- removed C17, C18, C21: C, Capacitor_SMD:C_0201_0603Metric, symbol Device:C
- removed U3: MAX-M8W-0, RocketClub:SMT_M8W-0_UBL, symbol Rocket Club 2025 Parts Symbols_Including_Full_Stm32:MAX-M8W-0
- added C14: 100nF, Capacitor_SMD:C_0201_0603Metric, symbol Device:C
- added C2: 47pF, symbol Device:C
- added C22: 1uF, Capacitor_SMD:C_0201_0603Metric, symbol Device:C
- added C27: 10nF, symbol Device:C
- added H1, H2, H3, H4: MountingHole_Pad_MP, symbol Mechanical:MountingHole_Pad_MP
- added J2: CNMHF1, symbol Group Rocket Symbol Library:CONMHF1-SMD-G-T
- added L1, L2, L4: BLM15HD102SN1D, IND_BLM15_0402_MUR, symbol Group Rocket Symbol Library:BLM15HD102SN1D
- added L3: 27nH, symbol Device:L
- added R1, R2: 10 Ohm, symbol Device:R
- added U2: MAX-M8W-0, SMT_M8W-0_UBL, symbol Group Rocket Symbol Library:MAX-M8W-0
- C10, C4: value C -> 10uF
- C11, C12, C13, C16, C19, C20, C3, C6, C8, C9: value C -> 100nF
- C7: value C -> 4.7uF
Connections:
- net 3.3V is gone; now on net +3.3V: C10.2, C11.2, C12.2, C15.2, C16.2, C19.2, C20.2, C23.1, C24.2, C25.1, C26.1, C3.2, C4.2, C5.2, C6.1, C7.1, C8.2, C9.2, IC1.13 (VDDA), IC1.19 (VDD_1), IC1.32 (VDD_2), IC1.48 (VDD_3), IC1.64 (VDD_4), IC2.17 (SA0/H_MOSI_), IC2.28 (VDDIO), IC2.3 (VDD), IC2.5 (PS1), IC4.12 (VCC_1), IC4.34 (VCC1_1), IC4.37 (VCC_2), IC4.39 (VCC1_2), Oscillator 3.3V 16MHz1.1 (VCTCXO), Oscillator 3.3V 16MHz1.4 (VDD), R3.1, R4.1, R5.1, U1.1 (VDD_IO), U1.14 (VDD), U1.8 (CS)
- net GND: now also C14.1, C22.1, C27.1, H1.MP, H2.MP, H3.MP, H4.MP, R2.2, U2.1 (GND), U2.12 (GND)
- net I2C1_SCL: now also U2.17 (SCL)
- net I2C1_SDA: now also U2.16 (SDA)
- net MAX_Reset: now also U2.9 (RESET_N)
- net +3.3V: now reaches IC1.1 (VBAT)
- net +3.3V: now also C14.2, C22.2, L4.1, L4.2
- new net: C27.2, L3.1, R1.1
- new net: L2.1, U2.2 (TxD)
- new net: L1.1, U2.3 (RxD)
- new net: C2.2, J2.1, L3.2
- new net: J2.S1, U2.10 (GND)
- new net: R2.1, U2.15 (V_ANT)
- new net: C2.1, U2.11 (RF_IN)
- new net +3.3V GPS: U2.6 (V_BCKP), U2.7 (VCC_IO), U2.8 (VCC)
- new net +5V: R1.2
- new net PPS: U2.4 (TIMEPULSE)
- new net Rx: L1.2
- new net Tx: L2.2
- no-connect marks 27 -> 23
Other:
- note added: "10 uF"
- note removed: "10 uF Aluminum"
- note removed: "GPS"
- moved on the sheet: C10
