File: KiCad Schematic and PCB/Rocket Club V1 Schematic I2C 9.kicad_sch (KiCad schematic)
At the start: 76 parts, among them IC1 STM32H573RIT6, IC4 MT29F1G08ABAEAWP_E, J1 5-146285-3, J2 CNMHF1, J3 6120XX21621_61201021621, J4 GSB1C4621DS2HR, Q1 2PD601BRL, SW2 CAS-D20TB, U1 H3LIS100DLTR, U2 MAX-M8W-0, U3 LSM6DSOTR, U4 NCV5662DSADJR4G, U5 LPS22HHTR, U6 AZ1084CD-3.3TRG1, U7 AZ1084CD-5.0TRG1, U8 USBLC6-2SC6, Y1 TSX-3225_16.0000MF09Z-AC6

Commit message: Finished schematic, will do a once over when I have more time
Parts:
- removed SW2: CAS-D20TB, symbol Group Rocket PCB Symbols:CAS-D20TB
- removed Y1: TSX-3225_16.0000MF09Z-AC6, symbol Group Rocket PCB Symbols:TSX-3225_16.0000MF09Z-AC6
- added C17, C33: C, symbol Device:C
- added D2, D3: LED, symbol Device:LED
- added R13, R16: R, symbol Device:R
- added R17: 100ohm, symbol Device:R
- added R18: 10Kohm, symbol Device:R
- added SW1: SW_SPDT_321, Group Rocket Main PCB:CL-SB-12B-02T, symbol Switch:SW_SPDT_321
- added SW2: MFS201N-9-Z, Group Rocket Main PCB:MFS201N-9-Z_NDC, symbol Group Rocket PCB Symbols:MFS201N-9-Z
- added U10: FDD306P, Group Rocket Main PCB:TO252-3_369AS_FAS, symbol Group Rocket PCB Symbols:FDD306P
- added U9: ~, symbol Group Rocket PCB Symbols:BAT_16GA_THT_PAD
- added Y2: ABM11W-48.0000MHZ-7-B1U-T3, symbol Group Rocket PCB Symbols:ABM11W-48.0000MHZ-7-B1U-T3
- C15, C32: value 8pF -> 4pF
- C23, C24, C25, C26: value C -> 100nF
Connections:
- net BOOT1 is gone; now on net BOOT0: R14.1
- net +3.3V: now also SW1.3 (A)
- net +BATT: now also U10.3
- net GND: now also J4.A1_B12 (GND_A), J4.B1_A12 (GND_B), J4.SH1 (SHIELD), J4.SH2 (SHIELD), J4.SH3 (SHIELD), J4.SH4 (SHIELD), C17.1, C33.2, R13.2, R16.1, SW1.1 (C), SW2.2, SW2.5, U9.2 (-), Y2.2 (GND), Y2.4 (GND)
- net at C5.1, R14.2: now also D2.2 (A), SW1.2 (B)
- net at J4.A4_B9 (VBUS_A), J4.B4_A9 (VBUS_B), U8.5: now also D3.2 (A)
- net at C32.1: now also IC1.6 (PH1-OSC_OUT), Y2.3; no longer IC1.4 (PC15-OSC32_OUT)
- net at C15.2: now also IC1.5 (PH0-OSC_IN), Y2.1; no longer IC1.3 (PC14-OSC32_IN)
- net at IC1.30 (VCAP_1): now also C33.1
- net at IC1.62 (VCAP_2): now also C17.2
- net KEY: no longer names the net of J3.7
- net NC: no longer names the net of J3.8
- new net: D3.1 (K), R16.2
- new net: R17.1, SW2.1, SW2.4
- new net: D2.1 (K), R13.1
- new net: R18.1, U10.2, U9.1 (+)
- new net: R17.2, R18.2, U10.1
- no-connect marks 15 -> 17
Other:
- note added: "3.3V Regulator"
- note added: "5V Regulator"
- note added: "Barometer"
- note added: "Boot Switch"
- note added: "Buzzer"
- note added: "GPS"
- note added: "Main Power FET and 16GA THT Terminal"
- note added: "NAND Flash"
- note added: "SOS Led"
- note added: "STM32H573RIT6 MAIN MCU"
- note added: "SWD/JTAG"
- note added: "Servo Power and Terminal"
- note added: "USB-C and TVS Diode"
- moved on the sheet: C13, C16, C18, C19, C2, C20, C21, C23, C24, C25, C26, C27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
